File: HydraODB/SchieldODB.brd (EAGLE design)
At the start: 59.9 x 37 mm, 6 parts, among them J1 HYDRABUS_SHIELD_CON_HEADER_2X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, J2 HYDRABUS_SHIELD_CON_HEADER_2X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, J3 HYDRABUS_SHIELD_CON_HEADER_2X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, U1 SN65HVD233D, U2 SN65HVD233D

Commit message: Schema and board corrections
Parts:
- added E$1: (no value), con-conrad:741256-49
- added E$2: (no value), ref-packages:RTRIMT93YA
- added E$3: (no value), v-reg:79XXS_
- moved U2 11.1 mm to (30.1, 11.9)
- moved U1 11.1 mm to (30.0, 22.6)
Changed lines of the file:
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@@
 <attribute name="NAME" x="36.83" y="25.7683" size="0.8128" layer="21" ratio="10"/>
 </element>
-<element name="U1" library="Texas Instruments_By_element14_Batch_1" package="SOIC127P600X175-8N" value="SN65HVD233D" x="41.021" y="22.352" rot="MR0">
-<attribute name="OC_NEWARK" value="54H4289" x="41.021" y="22.352" size="1.778" layer="28" rot="MR0" display="off"/>
-<attribute name="SUPPLIER" value="Texas Instruments" x="41.021" y="22.352" size="1.778" layer="28" rot="MR0" display="off"/>
-<attribute name="OC_FARNELL" value="1207268" x="41.021" y="22.352" size="1.778" layer="28" rot="MR0" display="off"/>
-<attribute name="PACKAGE" value="SOIC-8" x="41.021" y="22.352" size="1.778" layer="28" rot="MR0" display="off"/>
-<attribute name="MPN" value="SN65HVD233D" x="41.021" y="22.352" size="1.778" layer="28" rot="MR0" display="off"/>
+<element name="U1" library="Texas Instruments_By_element14_Batch_1" package="SOIC127P600X175-8N" value="SN65HVD233D" x="29.972" y="22.606" rot="MR0">
+<attribute name="OC_NEWARK" value="54H4289" x="29.972" y="22.606" size="1.778" layer="28" rot="MR0" display="off"/>
+<attribute name="SUPPLIER" value="Texas Instruments" x="29.972" y="22.606" size="1.778" layer="28" rot="MR0" display="off"/>
+<attribute name="OC_FARNELL" value="1207268" x="29.972" y="22.606" size="1.778" layer="28" rot="MR0" display="off"/>
+<attribute name="PACKAGE" value="SOIC-8" x="29.972" y="22.606" size="1.778" layer="28" rot="MR0" display="off"/>
+<attribute name="MPN" value="SN65HVD233D" x="29.972" y="22.606" size="1.778" layer="28" rot="MR0" display="off"/>
 </element>
-<element name="U2" library="Texas Instruments_By_element14_Batch_1" package="SOIC127P600X175-8N" value="SN65HVD233D" x="41.021" y="13.843" rot="MR0">
-<attribute name="OC_NEWARK" value="54H4289" x="41.021" y="13.843" size="1.778" layer="28" rot="MR0" display="off"/>
-<attribute name="SUPPLIER" value="Texas Instruments" x="41.021" y="13.843" size="1.778" layer="28" rot="MR0" display="off"/>
-<attribute name="OC_FARNELL" value="1207268" x="41.021" y="13.843" size="1.778" layer="28" rot="MR0" display="off"/>
-<attribute name="PACKAGE" value="SOIC-8" x="41.021" y="13.843" size="1.778" layer="28" rot="MR0" display="off"/>
-<attribute name="MPN" value="SN65HVD233D" x="41.021" y="13.843" size="1.778" layer="28" rot="MR0" display="off"/>
+<element name="U2" library="Texas Instruments_By_element14_Batch_1" package="SOIC127P600X175-8N" value="SN65HVD233D" x="30.099" y="11.938" rot="MR0">
+<attribute name="OC_NEWARK" value="54H4289" x="30.099" y="11.938" size="1.778" layer="28" rot="MR0" display="off"/>
+<attribute name="SUPPLIER" value="Texas Instruments" x="30.099" y="11.938" size="1.778" layer="28" rot="MR0" display="off"/>
+<attribute name="OC_FARNELL" value="1207268" x="30.099" y="11.938" size="1.778" layer="28" rot="MR0" display="off"/>
+<attribute name="PACKAGE" value="SOIC-8" x="30.099" y="11.938" size="1.778" layer="28" rot="MR0" display="off"/>
+<attribute name="MPN" value="SN65HVD233D" x="30.099" y="11.938" size="1.778" layer="28" rot="MR0" display="off"/>
 </element>
+<element name="E$1" library="con-conrad" package="741256-49" value="" x="3.175" y="18.034" rot="R90"/>
+<element name="E$2" library="ref-packages" package="RTRIMT93YA" value="" x="43.053" y="17.653"/>
+<element name="E$3" library="v-reg" package="79XXS_" value="" x="5.842" y="2.159" rot="R180"/>
 </elements>
 <signals>
@@
 <contactref element="SWD_DEBUG" pad="1"/>
 <contactref element="U2" pad="3"/>
+<wire x1="55.626" y1="26.162" x2="50.038" y2="33.782" width="0" layer="19" extent="1-1"/>
+<wire x1="37.338" y1="27.9908" x2="50.038" y2="33.782" width="0" layer="19" extent="1-1"/>
+<wire x1="50.038" y1="3.302" x2="55.626" y2="26.162" width="0" layer="19" extent="1-1"/>
+<wire x1="32.5628" y1="11.303" x2="37.338" y2="27.9908" width="0" layer="19" extent="16-16"/>
 </signal>
 <signal name="GND">
@@
 <contactref element="J3" pad="2"/>
 <contactref element="J2" pad="1"/>
+<wire x1="27.178" y1="3.302" x2="27.178" y2="33.782" width="0" layer="19" extent="1-1"/>
 </signal>
 <signal name="PB11">
