File: HydraODB/SchieldODB.sch (EAGLE design)
At the start: 8 parts, among them J1 HYDRABUS_SHIELD_CON_HEADER_2X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, J2 HYDRABUS_SHIELD_CON_HEADER_2X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, J3 HYDRABUS_SHIELD_CON_HEADER_2X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, U2 SN65HVD233D

Commit message: Schema and board corrections
Parts:
- added R1: (no value), pot:TRIM_EU-S64W
- added R2: (no value), pot:TRIM_EU-S63S
Connections:
- net PC8_SDIO_D0 renamed N$10
- removed net PB7: TRANSCEIVER1.CANH, X1-2.KL
- removed net PB8: J1.6, TRANSCEIVER1.CANL
- removed net PC10_SDIO_D2: J3.14
- removed net PC11_SDIO_D3: J3.12
- removed net PC9_SDIO_D1: J3.16
- new net N$4: J1.6, TRANSCEIVER1.D
- new net N$5: TRANSCEIVER1.R
- new net N$6: R1.S, U2.NC
- new net N$7: R2.S
- new net N$8: TRANSCEIVER1.CANL
- new net N$9: TRANSCEIVER1.CANH
- net GND: no longer TRANSCEIVER1.NC, U2.NC
- net N$2: no longer U2.CANL, X2-1.KL
- net PB6: no longer U2.CANH, X2-2.KL
Changed lines of the file:
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@@
 <part name="GND8" library="supply1" deviceset="GND" device=""/>
 <part name="GNDI1" library="supply1" deviceset="GNDI" device=""/>
+<part name="R1" library="pot" deviceset="TRIM_EU-" device="S64W"/>
+<part name="R2" library="pot" deviceset="TRIM_EU-" device="S63S"/>
 </parts>
 <sheets>
@@
 <instance part="GND8" gate="1" x="193.04" y="116.84"/>
 <instance part="GNDI1" gate="G$1" x="193.04" y="124.46"/>
+<instance part="R1" gate="1" x="104.14" y="76.2"/>
+<instance part="R2" gate="1" x="109.22" y="119.38"/>
 </instances>
 <busses>
@@
 <pinref part="TRANSCEIVER1" gate="A" pin="GND"/>
 <pinref part="GND2" gate="1" pin="GND"/>
-<pinref part="TRANSCEIVER1" gate="A" pin="NC"/>
-<wire x1="116.84" y1="124.46" x2="116.84" y2="119.38" width="0.1524" layer="91"/>
 <wire x1="116.84" y1="119.38" x2="116.84" y2="111.76" width="0.1524" layer="91"/>
 </segment>
@@
 <pinref part="GND7" gate="1" pin="GND"/>
 <wire x1="119.38" y1="76.2" x2="119.38" y2="71.12" width="0.1524" layer="91"/>
-<pinref part="U2" gate="A" pin="NC"/>
-<wire x1="119.38" y1="81.28" x2="119.38" y2="76.2" width="0.1524" layer="91"/>
 </segment>
 <segment>
@@
 </segment>
 </net>
-<net name="PB8" class="0">
-<segment>
-<pinref part="TRANSCEIVER1" gate="A" pin="CANL"/>
-<wire x1="152.4" y1="137.16" x2="165.1" y2="152.4" width="0.1524" layer="91"/>
-<wire x1="165.1" y1="152.4" x2="180.34" y2="152.4" width="0.1524" layer="91"/>
-<pinref part="J1" gate="J" pin="6"/>
-<wire x1="83.82" y1="129.54" x2="91.44" y2="137.16" width="0.1524" layer="91"/>
-<wire x1="91.44" y1="137.16" x2="152.4" y2="137.16" width="0.1524" layer="91"/>
-</segment>
-</net>
 <net name="BOOT0" class="0">
 <segment>
@@
 </segment>
 </net>
-<net name="PB7" class="0">
-<segment>
-<wire x1="83.82" y1="127" x2="81.28" y2="127" width="0.1524" layer="91"/>
-<pinref part="TRANSCEIVER1" gate="A" pin="CANH"/>
-<pinref part="X1" gate="-2" pin="KL"/>
-<wire x1="152.4" y1="134.62" x2="165.1" y2="147.32" width="0.1524" layer="91"/>
-<wire x1="165.1" y1="147.32" x2="185.42" y2="147.32" width="0.1524" layer="91"/>
-<wire x1="81.28" y1="127" x2="88.9" y2="134.62" width="0.1524" layer="91"/>
-<wire x1="88.9" y1="134.62" x2="152.4" y2="134.62" width="0.1524" layer="91"/>
-</segment>
-</net>
 <net name="PB6" class="0">
 <segment>
@@
 <label x="88.9" y="121.92" size="1.778" layer="95"/>
 <pinref part="J1" gate="J" pin="12"/>
-<pinref part="U2" gate="A" pin="CANH"/>
-<pinref part="X2" gate="-2" pin="KL"/>
-<wire x1="154.94" y1="91.44" x2="167.64" y2="104.14" width="0.1524" layer="91"/>
-<wire x1="167.64" y1="104.14" x2="187.96" y2="104.14" width="0.1524" layer="91"/>
-<wire x1="88.9" y1="121.92" x2="119.38" y2="91.44" width="0.1524" layer="91"/>
-<wire x1="119.38" y1="91.44" x2="154.94" y2="91.44" width="0.1524" layer="91"/>
 </segment>
 </net>
@@
 </segment>
 </net>
-<net name="PC9_SDIO_D1" class="0">
-<segment>
-<wire x1="-30.48" y1="109.22" x2="-25.4" y2="109.22" width="0.1524" layer="91"/>
-<label x="-25.4" y="109.22" size="1.778" layer="95"/>
-<pinref part="J3" gate="J" pin="16"/>
-</segment>
-</net>
-<net name="PC8_SDIO_D0" class="0">
-<segment>
-<wire x1="-30.48" y1="106.68" x2="-25.4" y2="106.68" width="0.1524" layer="91"/>
-<label x="-25.4" y="106.68" size="1.778" layer="95"/>
-<pinref part="J3" gate="J" pin="18"/>
-</segment>
-</net>
 <net name="PB2_BOOT1" class="0">
 <segment>
@@
 </segment>
 </net>
-<net name="PC11_SDIO_D3" class="0">
-<segment>
-<wire x1="-30.48" y1="114.3" x2="-25.4" y2="114.3" width="0.1524" layer="91"/>
-<label x="-25.4" y="114.3" size="1.778" layer="95"/>
-<pinref part="J3" gate="J" pin="12"/>
-</segment>
-</net>
-<net name="PC10_SDIO_D2" class="0">
-<segment>
-<wire x1="-30.48" y1="111.76" x2="-25.4" y2="111.76" width="0.1524" layer="91"/>
-<label x="-25.4" y="111.76" size="1.778" layer="95"/>
-<pinref part="J3" gate="J" pin="14"/>
-</segment>
-</net>
 <net name="N$1" class="0">
 <segment>
@@
 <net name="N$2" class="0">
 <segment>
-<pinref part="X2" gate="-1" pin="KL"/>
-<pinref part="U2" gate="A" pin="CANL"/>
 <pinref part="J1" gate="J" pin="10"/>
-<wire x1="83.82" y1="124.46" x2="93.98" y2="124.46" width="0.1524" layer="91"/>
-<wire x1="93.98" y1="124.46" x2="124.46" y2="93.98" width="0.1524" layer="91"/>
-<wire x1="124.46" y1="93.98" x2="154.94" y2="93.98" width="0.1524" layer="91"/>
-<wire x1="154.94" y1="93.98" x2="170.18" y2="109.22" width="0.1524" layer="91"/>
-<wire x1="170.18" y1="109.22" x2="187.96" y2="109.22" width="0.1524" layer="91"/>
+<wire x1="83.82" y1="124.46" x2="99.06" y2="124.46" width="0.1524" layer="91"/>
 <label x="99.06" y="124.46" size="1.778" layer="95"/>
 <label x="99.06" y="129.54" size="1.778" layer="95"/>
+<wire x1="99.06" y1="124.46" x2="101.6" y2="127" width="0.1524" layer="91"/>
+<wire x1="101.6" y1="127" x2="119.38" y2="127" width="0.1524" layer="91"/>
 </segment>
 </net>
@@
 </segment>
 </net>
+<net name="N$3" class="0">
+<segment>
+<wire x1="177.8" y1="109.22" x2="182.88" y2="109.22" width="0.1524" layer="91"/>
+</segment>
+</net>
+<net name="N$6" class="0">
+<segment>
+<pinref part="R1" gate="1" pin="S"/>
+<pinref part="U2" gate="A" pin="NC"/>
+<wire x1="109.22" y1="76.2" x2="114.3" y2="81.28" width="0.1524" layer="91"/>
+<wire x1="114.3" y1="81.28" x2="119.38" y2="81.28" width="0.1524" layer="91"/>
+</segment>
+</net>
+<net name="N$7" class="0">
+<segment>
+<pinref part="R2" gate="1" pin="S"/>
+<wire x1="114.3" y1="119.38" x2="116.84" y2="121.92" width="0.1524" layer="91"/>
+</segment>
+</net>
+<net name="N$8" class="0">
+<segment>
+<pinref part="TRANSCEIVER1" gate="A" pin="CANL"/>
+<wire x1="152.4" y1="137.16" x2="152.4" y2="152.4" width="0.1524" layer="91"/>
+<wire x1="152.4" y1="152.4" x2="180.34" y2="152.4" width="0.1524" layer="91"/>
+</segment>
+</net>
+<net name="N$5" class="0">
+<segment>
+<wire x1="83.82" y1="127" x2="93.98" y2="127" width="0.1524" layer="91"/>
+<pinref part="TRANSCEIVER1" gate="A" pin="R"/>
+<wire x1="152.4" y1="129.54" x2="93.98" y2="129.54" width="0.1524" layer="91"/>
+<wire x1="93.98" y1="129.54" x2="93.98" y2="127" width="0.1524" layer="91"/>
+</segment>
+</net>
+<net name="N$4" class="0">
+<segment>
+<pinref part="J1" gate="J" pin="6"/>
+<pinref part="TRANSCEIVER1" gate="A" pin="D"/>
+<wire x1="83.82" y1="129.54" x2="96.52" y2="132.08" width="0.1524" layer="91"/>
+<wire x1="96.52" y1="132.08" x2="116.84" y2="132.08" width="0.1524" layer="91"/>
+</segment>
+</net>
+<net name="N$9" class="0">
+<segment>
+<pinref part="TRANSCEIVER1" gate="A" pin="CANH"/>
+<wire x1="152.4" y1="134.62" x2="162.56" y2="147.32" width="0.1524" layer="91"/>
+<wire x1="162.56" y1="147.32" x2="180.34" y2="147.32" width="0.1524" layer="91"/>
+</segment>
+</net>
+<net name="N$10" class="0">
+<segment>
+<pinref part="J3" gate="J" pin="18"/>
+<wire x1="-30.48" y1="106.68" x2="-25.4" y2="106.68" width="0.1524" layer="91"/>
+<label x="-25.4" y="106.68" size="1.778" layer="95"/>
+</segment>
+</net>
 </nets>
 </sheet>
 </sheets>
+<errors>
+</errors>
 </schematic>
 </drawing>

Commit message: VReg add, CanBus 2 rewired
Parts:
- added IC1: 7805L, linear:7805L
Connections:
- new net N$11: U2.CANH
- new net N$13: IC1.VI
- new net N$3: U2.CANL
- net +3V3: now also R1.E, R2.E
- net GND: now also IC1.GND, R1.A, R2.A
Other:
- moved on the sheet: R2
Changed lines of the file:
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@@
 <part name="R1" library="pot" deviceset="TRIM_EU-" device="S64W"/>
 <part name="R2" library="pot" deviceset="TRIM_EU-" device="S63S"/>
+<part name="+3V6" library="supply1" deviceset="+3V3" device=""/>
+<part name="+3V8" library="supply1" deviceset="+3V3" device=""/>
+<part name="GND10" library="supply1" deviceset="GND" device=""/>
+<part name="GND11" library="supply1" deviceset="GND" device=""/>
+<part name="IC1" library="linear" deviceset="78*" device="L" technology="05"/>
+<part name="GND12" library="supply1" deviceset="GND" device=""/>
 </parts>
 <sheets>
@@
 <wire x1="125.73" y1="139.7" x2="118.11" y2="132.08" width="0.4064" layer="108"/>
 <text x="-50.8" y="142.24" size="1.778" layer="97">HydraBus Headers</text>
+<wire x1="121.92" y1="83.82" x2="119.38" y2="86.36" width="0.1524" layer="101"/>
+<wire x1="119.38" y1="86.36" x2="109.22" y2="86.36" width="0.1524" layer="101"/>
+<wire x1="109.22" y1="86.36" x2="99.06" y2="96.52" width="0.1524" layer="101"/>
+<wire x1="99.06" y1="96.52" x2="99.06" y2="104.14" width="0.1524" layer="101"/>
+<wire x1="99.06" y1="104.14" x2="93.98" y2="109.22" width="0.1524" layer="101"/>
+<wire x1="93.98" y1="109.22" x2="43.18" y2="109.22" width="0.1524" layer="101"/>
+<wire x1="43.18" y1="109.22" x2="43.18" y2="134.62" width="0.1524" layer="101"/>
+<wire x1="43.18" y1="134.62" x2="76.2" y2="134.62" width="0.1524" layer="101"/>
 </plain>
 <instances>
@@
 <instance part="TRANSCEIVER1" gate="A" x="134.62" y="132.08"/>
 <instance part="+3V1" gate="G$1" x="116.84" y="144.78"/>
-<instance part="GND2" gate="1" x="116.84" y="109.22"/>
+<instance part="GND2" gate="1" x="116.84" y="114.3"/>
 <instance part="U2" gate="A" x="137.16" y="88.9"/>
 <instance part="+3V3" gate="G$1" x="119.38" y="99.06"/>
@@
 <instance part="GNDI1" gate="G$1" x="193.04" y="124.46"/>
 <instance part="R1" gate="1" x="104.14" y="76.2"/>
-<instance part="R2" gate="1" x="109.22" y="119.38"/>
+<instance part="R2" gate="1" x="111.76" y="119.38"/>
+<instance part="+3V6" gate="G$1" x="111.76" y="124.46"/>
+<instance part="+3V8" gate="G$1" x="104.14" y="86.36"/>
+<instance part="GND10" gate="1" x="104.14" y="66.04"/>
+<instance part="GND11" gate="1" x="111.76" y="114.3"/>
+<instance part="IC1" gate="A1" x="165.1" y="60.96"/>
+<instance part="GND12" gate="1" x="165.1" y="50.8"/>
 </instances>
 <busses>
@@
 <pinref part="+3V3" gate="G$1" pin="+3V3"/>
 <wire x1="119.38" y1="93.98" x2="119.38" y2="96.52" width="0.1524" layer="91"/>
+</segment>
+<segment>
+<pinref part="R2" gate="1" pin="E"/>
+<pinref part="+3V6" gate="G$1" pin="+3V3"/>
+<wire x1="111.76" y1="121.92" x2="111.76" y2="124.46" width="0.1524" layer="91"/>
+</segment>
+<segment>
+<pinref part="R1" gate="1" pin="E"/>
+<pinref part="+3V8" gate="G$1" pin="+3V3"/>
+<wire x1="104.14" y1="81.28" x2="104.14" y2="83.82" width="0.1524" layer="91"/>
 </segment>
 </net>
@@
 <pinref part="TRANSCEIVER1" gate="A" pin="GND"/>
 <pinref part="GND2" gate="1" pin="GND"/>
-<wire x1="116.84" y1="119.38" x2="116.84" y2="111.76" width="0.1524" layer="91"/>
+<wire x1="116.84" y1="119.38" x2="116.84" y2="116.84" width="0.1524" layer="91"/>
 </segment>
 <segment>
@@
 <wire x1="193.04" y1="119.38" x2="190.5" y2="116.84" width="0.1524" layer="91"/>
 <wire x1="190.5" y1="116.84" x2="185.42" y2="116.84" width="0.1524" layer="91"/>
+</segment>
+<segment>
+<pinref part="R2" gate="1" pin="A"/>
+<pinref part="GND11" gate="1" pin="GND"/>
+<wire x1="111.76" y1="114.3" x2="111.76" y2="116.84" width="0.1524" layer="91"/>
+</segment>
+<segment>
+<pinref part="R1" gate="1" pin="A"/>
+<pinref part="GND10" gate="1" pin="GND"/>
+<wire x1="104.14" y1="71.12" x2="104.14" y2="68.58" width="0.1524" layer="91"/>
+</segment>
+<segment>
+<pinref part="GND12" gate="1" pin="GND"/>
+<pinref part="IC1" gate="A1" pin="GND"/>
 </segment>
 </net>
@@
 <net name="N$3" class="0">
 <segment>
-<wire x1="177.8" y1="109.22" x2="182.88" y2="109.22" width="0.1524" layer="91"/>
+<pinref part="U2" gate="A" pin="CANL"/>
+<wire x1="154.94" y1="93.98" x2="154.94" y2="109.22" width="0.1524" layer="91"/>
+<wire x1="154.94" y1="109.22" x2="182.88" y2="109.22" width="0.1524" layer="91"/>
 </segment>
 </net>
@@
 <segment>
 <pinref part="R2" gate="1" pin="S"/>
-<wire x1="114.3" y1="119.38" x2="116.84" y2="121.92" width="0.1524" layer="91"/>
+<wire x1="116.84" y1="119.38" x2="116.84" y2="124.46" width="0.1524" layer="91"/>
 </segment>
 </net>
@@
 </segment>
 </net>
+<net name="N$11" class="0">
+<segment>
+<pinref part="U2" gate="A" pin="CANH"/>
+<wire x1="154.94" y1="91.44" x2="165.1" y2="104.14" width="0.1524" layer="91"/>
+<wire x1="165.1" y1="104.14" x2="182.88" y2="104.14" width="0.1524" layer="91"/>
+</segment>
+</net>
+<net name="N$13" class="0">
+<segment>
+<pinref part="IC1" gate="A1" pin="VI"/>
+<wire x1="154.94" y1="60.96" x2="152.4" y2="83.82" width="0.1524" layer="91"/>
+<wire x1="152.4" y1="83.82" x2="185.42" y2="83.82" width="0.1524" layer="91"/>
+</segment>
+</net>

Commit message: Schema redisign
Connections:
- net PB1: now also U2.R
Other:
- moved on the sheet: IC1
Changed lines of the file:
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@@
 <wire x1="125.73" y1="139.7" x2="118.11" y2="132.08" width="0.4064" layer="108"/>
 <text x="-50.8" y="142.24" size="1.778" layer="97">HydraBus Headers</text>
-<wire x1="121.92" y1="83.82" x2="119.38" y2="86.36" width="0.1524" layer="101"/>
-<wire x1="119.38" y1="86.36" x2="109.22" y2="86.36" width="0.1524" layer="101"/>
-<wire x1="109.22" y1="86.36" x2="99.06" y2="96.52" width="0.1524" layer="101"/>
-<wire x1="99.06" y1="96.52" x2="99.06" y2="104.14" width="0.1524" layer="101"/>
-<wire x1="99.06" y1="104.14" x2="93.98" y2="109.22" width="0.1524" layer="101"/>
-<wire x1="93.98" y1="109.22" x2="43.18" y2="109.22" width="0.1524" layer="101"/>
-<wire x1="43.18" y1="109.22" x2="43.18" y2="134.62" width="0.1524" layer="101"/>
-<wire x1="43.18" y1="134.62" x2="76.2" y2="134.62" width="0.1524" layer="101"/>
 </plain>
 <instances>
@@
 <instance part="GND10" gate="1" x="104.14" y="66.04"/>
 <instance part="GND11" gate="1" x="111.76" y="114.3"/>
-<instance part="IC1" gate="A1" x="165.1" y="60.96"/>
-<instance part="GND12" gate="1" x="165.1" y="50.8"/>
+<instance part="IC1" gate="A1" x="187.96" y="63.5"/>
+<instance part="GND12" gate="1" x="187.96" y="50.8"/>
 </instances>
 <busses>
@@
 <pinref part="GND12" gate="1" pin="GND"/>
 <pinref part="IC1" gate="A1" pin="GND"/>
+<wire x1="187.96" y1="55.88" x2="187.96" y2="53.34" width="0.1524" layer="91"/>
 </segment>
 </net>
@@
 <segment>
 <wire x1="83.82" y1="132.08" x2="88.9" y2="132.08" width="0.1524" layer="91"/>
-<label x="88.9" y="132.08" size="1.778" layer="95"/>
 <pinref part="J1" gate="J" pin="4"/>
 </segment>
@@
 <net name="PB1" class="0">
 <segment>
-<wire x1="76.2" y1="132.08" x2="71.12" y2="132.08" width="0.1524" layer="91"/>
 <label x="71.12" y="132.08" size="1.778" layer="95" rot="R180"/>
 <pinref part="J1" gate="J" pin="3"/>
+<pinref part="U2" gate="A" pin="R"/>
+<wire x1="154.94" y1="86.36" x2="160.02" y2="86.36" width="0.1524" layer="91"/>
+<wire x1="160.02" y1="86.36" x2="160.02" y2="48.26" width="0.1524" layer="91"/>
+<wire x1="160.02" y1="48.26" x2="43.18" y2="48.26" width="0.1524" layer="91"/>
+<wire x1="43.18" y1="48.26" x2="43.18" y2="132.08" width="0.1524" layer="91"/>
+<wire x1="43.18" y1="132.08" x2="76.2" y2="132.08" width="0.1524" layer="91"/>
 </segment>
 </net>
 <net name="PB0" class="0">
 <segment>
-<wire x1="76.2" y1="134.62" x2="63.5" y2="134.62" width="0.1524" layer="91"/>
 <label x="63.5" y="134.62" size="1.778" layer="95" rot="R180"/>
 <pinref part="J1" gate="J" pin="1"/>
+<wire x1="76.2" y1="134.62" x2="45.72" y2="134.62" width="0.1524" layer="91"/>
+<wire x1="45.72" y1="134.62" x2="45.72" y2="109.22" width="0.1524" layer="91"/>
+<wire x1="45.72" y1="109.22" x2="109.22" y2="109.22" width="0.1524" layer="91"/>
+<wire x1="109.22" y1="109.22" x2="109.22" y2="88.9" width="0.1524" layer="91"/>
+<wire x1="109.22" y1="88.9" x2="124.46" y2="88.9" width="0.1524" layer="91"/>
 </segment>
 </net>
@@
 <net name="PB2_BOOT1" class="0">
 <segment>
-<wire x1="76.2" y1="129.54" x2="63.5" y2="129.54" width="0.1524" layer="91"/>
+<wire x1="76.2" y1="129.54" x2="66.04" y2="129.54" width="0.1524" layer="91"/>
 <label x="49.53" y="129.54" size="1.778" layer="95"/>
 <pinref part="J1" gate="J" pin="5"/>
+<wire x1="66.04" y1="129.54" x2="63.5" y2="129.54" width="0.1524" layer="91"/>
+<wire x1="121.92" y1="83.82" x2="106.68" y2="83.82" width="0.1524" layer="91"/>
+<wire x1="106.68" y1="83.82" x2="106.68" y2="96.52" width="0.1524" layer="91"/>
+<wire x1="106.68" y1="96.52" x2="96.52" y2="96.52" width="0.1524" layer="91"/>
+<wire x1="96.52" y1="96.52" x2="96.52" y2="53.34" width="0.1524" layer="91"/>
+<wire x1="96.52" y1="53.34" x2="40.64" y2="53.34" width="0.1524" layer="91"/>
+<wire x1="40.64" y1="53.34" x2="40.64" y2="129.54" width="0.1524" layer="91"/>
+<wire x1="40.64" y1="129.54" x2="63.5" y2="129.54" width="0.1524" layer="91"/>
 </segment>
 </net>
@@
 <net name="N$4" class="0">
 <segment>
+<pinref part="TRANSCEIVER1" gate="A" pin="D"/>
+<wire x1="91.44" y1="132.08" x2="116.84" y2="132.08" width="0.1524" layer="91"/>
+<wire x1="91.44" y1="132.08" x2="91.44" y2="129.54" width="0.1524" layer="91"/>
 <pinref part="J1" gate="J" pin="6"/>
-<pinref part="TRANSCEIVER1" gate="A" pin="D"/>
-<wire x1="83.82" y1="129.54" x2="96.52" y2="132.08" width="0.1524" layer="91"/>
-<wire x1="96.52" y1="132.08" x2="116.84" y2="132.08" width="0.1524" layer="91"/>
-</segment>
-</net>
-<net name="N$9" class="0">
-<segment>
-<pinref part="TRANSCEIVER1" gate="A" pin="CANH"/>
-<wire x1="152.4" y1="134.62" x2="162.56" y2="147.32" width="0.1524" layer="91"/>
-<wire x1="162.56" y1="147.32" x2="180.34" y2="147.32" width="0.1524" layer="91"/>
+<wire x1="83.82" y1="129.54" x2="91.44" y2="129.54" width="0.1524" layer="91"/>
 </segment>
 </net>
@@
 </segment>
 </net>
+<net name="N$9" class="0">
+<segment>
+<pinref part="TRANSCEIVER1" gate="A" pin="CANH"/>
+<wire x1="152.4" y1="134.62" x2="162.56" y2="134.62" width="0.1524" layer="91"/>
+<wire x1="162.56" y1="134.62" x2="162.56" y2="147.32" width="0.1524" layer="91"/>
+<wire x1="162.56" y1="147.32" x2="180.34" y2="147.32" width="0.1524" layer="91"/>
+</segment>
+</net>
 <net name="N$11" class="0">
 <segment>
 <pinref part="U2" gate="A" pin="CANH"/>
-<wire x1="154.94" y1="91.44" x2="165.1" y2="104.14" width="0.1524" layer="91"/>
-<wire x1="165.1" y1="104.14" x2="182.88" y2="104.14" width="0.1524" layer="91"/>
-</segment>
-</net>
-<net name="N$13" class="0">
+<wire x1="154.94" y1="91.44" x2="160.02" y2="91.44" width="0.1524" layer="91"/>
+<wire x1="160.02" y1="91.44" x2="160.02" y2="104.14" width="0.1524" layer="91"/>
+<wire x1="160.02" y1="104.14" x2="182.88" y2="104.14" width="0.1524" layer="91"/>
+</segment>
+</net>
+<net name="N$12" class="0">
 <segment>
 <pinref part="IC1" gate="A1" pin="VI"/>
-<wire x1="154.94" y1="60.96" x2="152.4" y2="83.82" width="0.1524" layer="91"/>
-<wire x1="152.4" y1="83.82" x2="185.42" y2="83.82" width="0.1524" layer="91"/>
-</segment>
-</net>
+<wire x1="177.8" y1="63.5" x2="172.72" y2="63.5" width="0.1524" layer="91"/>
+<wire x1="172.72" y1="63.5" x2="172.72" y2="83.82" width="0.1524" layer="91"/>
+<wire x1="172.72" y1="83.82" x2="180.34" y2="83.82" width="0.1524" layer="91"/>
+</segment>
+</net>
