File: HydraODB/OBDShield.sch (EAGLE design)
At the start: 30 parts, among them IC1 LM317MABDT, J1 HYDRABUS_SHIELD_CON_HEADER_2X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, J2 HYDRABUS_SHIELD_CON_HEADER_2X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, J3 HYDRABUS_SHIELD_CON_HEADER_2X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, K1 TS-1101F, U1 SN65HVD233DG4, U2 SN65HVD233DG4

Commit message: Decap condos
Parts:
- JP1: value (none) -> H1
- R10: value (none) -> 470
Connections:
- net N$10 renamed CAN1H
- net N$11 renamed CAN2L
- net N$12 renamed CAN2H
- net N$9 renamed CAN1L
- removed net N$15: R3.2
- net VUSB: now also R3.2
Other:
- moved on the sheet: C1, LPWR, R3
Changed lines of the file:
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@@
 <part name="GND16" library="supply1" deviceset="GND" device=""/>
 <part name="GND17" library="supply1" deviceset="GND" device=""/>
-<part name="JP1" library="jumper" deviceset="JP1E" device=""/>
+<part name="JP1" library="jumper" deviceset="JP1E" device="" value="H1"/>
 <part name="JP2" library="jumper" deviceset="JP1E" device=""/>
 <part name="K1" library="Seeed-OPL-Button" deviceset="DIP-BUTTON-FRONT-WHITE(2P-3.4X6MM)" device="" value="TS-1101F"/>
@@
 <part name="+3V6" library="supply1" deviceset="+3V3" device=""/>
 <part name="GND20" library="supply1" deviceset="GND" device=""/>
-<part name="R10" library="resistor" deviceset="R-EU_" device="R0603"/>
+<part name="R10" library="resistor" deviceset="R-EU_" device="R0603" value="470"/>
 <part name="R11" library="resistor" deviceset="R-EU_" device="R0603"/>
 </parts>
@@
 <instance part="R1" gate="1" x="142.24" y="96.52"/>
 <instance part="R2" gate="1" x="147.32" y="30.48"/>
-<instance part="VUSB2" gate="G$1" x="1.524" y="91.44"/>
+<instance part="VUSB2" gate="G$1" x="1.524" y="93.98"/>
 <instance part="+3V1" gate="G$1" x="160.02" y="45.72"/>
 <instance part="GND2" gate="1" x="142.24" y="83.82"/>
 <instance part="+3V3" gate="G$1" x="157.48" y="140.97"/>
 <instance part="SV1" gate="G$1" x="215.9" y="91.44" rot="R180"/>
-<instance part="GND7" gate="1" x="-12.7" y="62.484" rot="MR0"/>
+<instance part="GND7" gate="1" x="-12.7" y="63.754" rot="MR0"/>
 <instance part="P+1" gate="1" x="-22.86" y="96.52"/>
 <instance part="P+2" gate="1" x="210.82" y="73.66" rot="R270"/>
@@
 <instance part="GND11" gate="1" x="130.81" y="97.79" rot="MR0"/>
 <instance part="GND12" gate="1" x="153.67" y="13.97" rot="MR0"/>
-<instance part="LPWR" gate="G$1" x="-2.54" y="73.66"/>
+<instance part="LPWR" gate="G$1" x="1.524" y="73.152"/>
 <instance part="LRXCAN1" gate="G$1" x="124.46" y="147.32" rot="R180"/>
 <instance part="LTXCAN1" gate="G$1" x="132.08" y="147.32" rot="R180"/>
 <instance part="LRXCAN2" gate="G$1" x="127" y="66.04" rot="R180"/>
 <instance part="LTXCAN2" gate="G$1" x="134.62" y="66.04" rot="R180"/>
-<instance part="R3" gate="G$1" x="-2.54" y="83.82" rot="R90"/>
+<instance part="R3" gate="G$1" x="1.524" y="86.36" rot="R90"/>
 <instance part="R4" gate="G$1" x="124.46" y="134.62" rot="R90"/>
 <instance part="R5" gate="G$1" x="132.08" y="134.62" rot="R90"/>
@@
 <instance part="GND15" gate="1" x="125.73" y="82.55" rot="MR180"/>
 <instance part="GND16" gate="1" x="133.35" y="82.55" rot="MR180"/>
-<instance part="GND17" gate="1" x="-2.54" y="62.484" rot="MR0"/>
+<instance part="GND17" gate="1" x="1.524" y="63.246" rot="MR0"/>
 <instance part="JP1" gate="A" x="144.78" y="142.24"/>
 <instance part="JP2" gate="A" x="149.86" y="63.5"/>
 <instance part="K1" gate="G$1" x="48.26" y="48.26" rot="R270"/>
-<instance part="C1" gate="G$1" x="-22.86" y="81.28" rot="R270"/>
+<instance part="C1" gate="G$1" x="-22.86" y="83.82" rot="R270"/>
 <instance part="C2" gate="G$1" x="160.02" y="55.88" rot="R270"/>
 <instance part="C3" gate="G$1" x="165.1" y="132.08" rot="R270"/>
@@
 </segment>
 <segment>
-<pinref part="GND8" gate="1" pin="GND"/>
-<pinref part="SV1" gate="G$1" pin="5"/>
-<wire x1="203.2" y1="83.82" x2="203.2" y2="88.9" width="0.1524" layer="91"/>
-<wire x1="203.2" y1="88.9" x2="208.28" y2="88.9" width="0.1524" layer="91"/>
-</segment>
-<segment>
 <pinref part="U1" gate="A" pin="LBK"/>
 <wire x1="157.48" y1="104.14" x2="130.81" y2="104.14" width="0.1524" layer="91"/>
@@
 <wire x1="-12.7" y1="83.82" x2="-12.7" y2="76.2" width="0.1524" layer="91"/>
 <pinref part="GND7" gate="1" pin="GND"/>
-<wire x1="-12.7" y1="76.2" x2="-12.7" y2="65.024" width="0.1524" layer="91"/>
+<wire x1="-12.7" y1="76.2" x2="-12.7" y2="66.294" width="0.1524" layer="91"/>
 <wire x1="-22.86" y1="76.2" x2="-12.7" y2="76.2" width="0.1524" layer="91"/>
 <junction x="-12.7" y="76.2"/>
 <junction x="-22.86" y="76.2"/>
-<wire x1="-22.86" y1="76.2" x2="-22.86" y2="77.47" width="0.1524" layer="91"/>
+<wire x1="-22.86" y1="76.2" x2="-22.86" y2="80.01" width="0.1524" layer="91"/>
 <pinref part="C1" gate="G$1" pin="2"/>
 </segment>
@@
 <segment>
 <pinref part="LPWR" gate="G$1" pin="C"/>
-<wire x1="-2.54" y1="68.58" x2="-2.54" y2="65.024" width="0.1524" layer="91"/>
+<wire x1="1.524" y1="68.072" x2="1.524" y2="65.786" width="0.1524" layer="91"/>
 <pinref part="GND17" gate="1" pin="GND"/>
 </segment>
@@
 <junction x="160.02" y="62.992"/>
 </segment>
+<segment>
+<pinref part="GND8" gate="1" pin="GND"/>
+<pinref part="SV1" gate="G$1" pin="5"/>
+<wire x1="203.2" y1="83.82" x2="203.2" y2="88.9" width="0.1524" layer="91"/>
+<wire x1="203.2" y1="88.9" x2="208.28" y2="88.9" width="0.1524" layer="91"/>
+</segment>
 </net>
 <net name="SWD_SWDIO" class="0">
@@
 <segment>
 <pinref part="IC1" gate="G$1" pin="OUT"/>
-<wire x1="-5.08" y1="91.44" x2="-2.54" y2="91.44" width="0.1524" layer="91"/>
+<wire x1="-5.08" y1="91.44" x2="1.524" y2="91.44" width="0.1524" layer="91"/>
 <pinref part="VUSB2" gate="G$1" pin="VUSB"/>
-<junction x="-2.54" y="91.44"/>
-<wire x1="-2.54" y1="91.44" x2="1.524" y2="91.44" width="0.1524" layer="91"/>
+<junction x="1.524" y="91.44"/>
+<wire x1="1.524" y1="91.44" x2="1.524" y2="93.98" width="0.1524" layer="91"/>
 <junction x="-5.08" y="91.44"/>
+<pinref part="R3" gate="G$1" pin="2"/>
 </segment>
 </net>
@@
 </segment>
 </net>
-<net name="N$10" class="0">
+<net name="CAN1H" class="0">
 <segment>
 <pinref part="SV1" gate="G$1" pin="2"/>
@@
 </segment>
 </net>
-<net name="N$11" class="0">
+<net name="CAN2L" class="0">
 <segment>
 <pinref part="U2" gate="A" pin="CANL"/>
@@
 <junction x="-22.86" y="91.44"/>
 <pinref part="C1" gate="G$1" pin="1"/>
-<wire x1="-22.86" y1="85.09" x2="-22.86" y2="91.44" width="0.1524" layer="91"/>
+<wire x1="-22.86" y1="87.63" x2="-22.86" y2="91.44" width="0.1524" layer="91"/>
 </segment>
 <segment>
@@
 <pinref part="LPWR" gate="G$1" pin="A"/>
 <pinref part="R3" gate="G$1" pin="1"/>
-<wire x1="-2.54" y1="78.74" x2="-2.54" y2="76.2" width="0.1524" layer="91"/>
-<junction x="-2.54" y="78.74"/>
-<junction x="-2.54" y="76.2"/>
-</segment>
-</net>
-<net name="N$15" class="0">
-<segment>
-<pinref part="R3" gate="G$1" pin="2"/>
-<wire x1="-2.54" y1="88.9" x2="-2.54" y2="90.932" width="0.1524" layer="91"/>
-<junction x="-2.54" y="88.9"/>
+<wire x1="1.524" y1="81.28" x2="1.524" y2="75.692" width="0.1524" layer="91"/>
+<junction x="1.524" y="81.28"/>
+<junction x="1.524" y="75.692"/>
 </segment>
 </net>
@@
 </segment>
 </net>
-<net name="N$9" class="0">
+<net name="CAN1L" class="0">
 <segment>
 <pinref part="SV1" gate="G$1" pin="1"/>
@@
 </segment>
 </net>
-<net name="N$12" class="0">
+<net name="CAN2H" class="0">
 <segment>
 <pinref part="U2" gate="A" pin="CANH"/>
